File: PCB/rev1.0/0xcb-static.kicad_pcb (KiCad board)
At the start: 2 copper layers, 223.8 x 108.2 mm, 126 parts, among them J1 USB_C_Receptacle_USB2.0, J2 AVR-ISP-6, SW1 RESET, SW2 BOOT, U1 ATmega328-P, Y1 16MHz

Commit message: added v1
Parts:
- removed the L2 at (229.1, 64.6)
- added L1: LOGO, static:logo, F.Cu at (232.5, 64.3)
- L3: renamed from G***; footprint LOGO -> static:LOGO
- MX1, MX10, MX11, MX14, MX15, MX16, MX17, MX18, MX19, MX2, MX20, MX21, MX22, MX24, MX26, MX27, MX28, MX29, MX3, MX30, MX31, MX32, MX33, MX34, MX36, MX37, MX37_2, MX38, MX38_2, MX4, MX40, MX40_1, MX42, MX43, MX44, MX5, MX6, MX7, MX8, MX9: footprint MX_Only:MXOnly-1U-NoLED -> static:MXOnly-1U-NoLED
- MX13, MX35, MX36_1, MX37_1, MX38_1, MX43_1, MX44_1: footprint MX_Only:MXOnly-1.25U-NoLED -> static:MXOnly-1.25U-NoLED
- MX23, MX25: footprint MX_Only:MXOnly-1.75U-NoLED -> static:MXOnly-1.75U-NoLED
- MX39, MX41_1: footprint MX_Only:MXOnly-2.75U-NoLED -> static:MXOnly-2.75U-NoLED
- MX39_1, MX41: footprint MX_Only:MXOnly-2.25U-NoLED -> static:MXOnly-2.25U-NoLED
- MX40_2: footprint MX_Only:MXOnly-6.25U-NoLED -> static:MXOnly-6.25U-NoLED
- renumbered L1 to L2
