File: PCB/rev1.0/0xcb-static.kicad_sch (KiCad schematic)
At the start: 112 parts, among them J1 USB_C_Receptacle_USB2.0, J2 AVR-ISP-6, SW1 RESET, SW2 BOOT, U1 ATmega328-P, Y1 16MHz

Commit message: added v1
Parts:
- C1, C2: Part Nb. (none) -> C277965
- C3, C4: Part Nb. (none) -> C254096
- D1, D10, D11, D12, D13, D14, D15, D16, D17, D18, D19, D2, D20, D21, D22, D23, D24, D25, D26, D27, D28, D29, D3, D30, D31, D32, D33, D34, D35, D36, D37, D38, D39, D4, D40, D41, D42, D43, D44, D45, D48, D49, D5, D50, D6, D7, D8, D9: Part Nb. (none) -> C14538
- D46, D47: Part Nb. (none) -> C2532
- F1: Part Nb. (none) -> C268799
- J1: Part Nb. (none) -> 2073-USB4085-GF-ACT-ND
- J2: Part Nb. (none) -> -; now left out of the parts list
- MX1, MX10, MX11, MX13, MX14, MX15, MX16, MX17, MX18, MX19, MX2, MX20, MX21, MX22, MX23, MX24, MX25, MX26, MX27, MX28, MX29, MX3, MX30, MX31, MX32, MX33, MX34, MX35, MX36, MX37, MX38, MX39, MX4, MX40, MX41, MX42, MX43, MX44, MX5, MX6, MX7, MX8, MX9: symbol MX_Alps_Hybrid:MX-NoLED -> static:MX-NoLED; Part Nb. (none) -> amz
- MX12: Part Nb. (none) -> amz
- OL1: symbol kbd:OLED -> static:OLED; Part Nb. (none) -> amz
- R1, R2: Part Nb. (none) -> C58676
- R3, R4: Part Nb. (none) -> C713897
- R5: Part Nb. (none) -> C58673
- R6: Part Nb. (none) -> C433494
- SW1, SW2: Part Nb. (none) -> C127509
- U1: Part Nb. (none) -> C613508
- Y1: Part Nb. (none) -> C16212

Commit message: updated prod files
Parts:
- renumbered D48 to D46, D49 to D47, D50 to D48, D46 to D49, D47 to D50
Connections:
- net COL0: now also J2.3 (SCK)
- net ROW5: no longer J2.4 (MOSI)
- net ROW6: now also J2.4 (MOSI); no longer J2.1 (MISO)
- net ROW7: now also J2.1 (MISO); no longer J2.3 (SCK)
Changed lines of the file:
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@@
-(kicad_sch (version 20210406) (generator eeschema)
+(kicad_sch (version 20210621) (generator eeschema)
   (paper "A4")
   (title_block
@@
     )
   )
-  (global_label "ROW6" (shape input) (at 129.54 161.29 0) (fields_autoplaced)
+  (global_label "ROW7" (shape input) (at 129.54 161.29 0) (fields_autoplaced)
     (effects (font (size 1.27 1.27)) (justify left))
-    (property "Intersheet References" "${INTERSHEET_REFS}" (id 0) (at 137.2145 161.3694 0)
+    (property "Intersheet References" "${INTERSHEET_REFS}" (id 0) (at 137.2145 161.2106 0)
       (effects (font (size 1.27 1.27)) (justify left) hide)
     )
   )
-  (global_label "ROW5" (shape input) (at 129.54 163.83 0) (fields_autoplaced)
+  (global_label "ROW6" (shape input) (at 129.54 163.83 0) (fields_autoplaced)
     (effects (font (size 1.27 1.27)) (justify left))
-    (property "Intersheet References" "${INTERSHEET_REFS}" (id 0) (at 137.2145 163.9094 0)
+    (property "Intersheet References" "${INTERSHEET_REFS}" (id 0) (at 137.2145 163.7506 0)
       (effects (font (size 1.27 1.27)) (justify left) hide)
     )
   )
-  (global_label "ROW7" (shape input) (at 129.54 166.37 0) (fields_autoplaced)
+  (global_label "COL0" (shape input) (at 129.54 166.37 0) (fields_autoplaced)
     (effects (font (size 1.27 1.27)) (justify left))
-    (property "Intersheet References" "${INTERSHEET_REFS}" (id 0) (at 137.2145 166.4494 0)
+    (property "Intersheet References" "${INTERSHEET_REFS}" (id 0) (at 136.7912 166.2906 0)
       (effects (font (size 1.27 1.27)) (justify left) hide)
     )
@@
   (symbol (lib_id "Device:D_Schottky") (at 46.99 45.72 270) (unit 1)
     (in_bom yes) (on_board yes) (fields_autoplaced)
-    (property "Reference" "D46" (id 0) (at 49.53 45.0849 90)
+    (property "Reference" "D49" (id 0) (at 49.53 45.0849 90)
       (effects (font (size 1.27 1.27)) (justify left))
     )
@@
   (symbol (lib_id "Device:D_Schottky") (at 59.69 45.72 270) (unit 1)
     (in_bom yes) (on_board yes) (fields_autoplaced)
-    (property "Reference" "D47" (id 0) (at 62.23 45.0849 90)
+    (property "Reference" "D50" (id 0) (at 62.23 45.0849 90)
       (effects (font (size 1.27 1.27)) (justify left))
     )
@@
   (symbol (lib_id "Diode:1N4148") (at 231.14 113.03 90) (unit 1)
     (in_bom yes) (on_board yes)
-    (property "Reference" "D48" (id 0) (at 226.06 112.3949 90)
+    (property "Reference" "D46" (id 0) (at 226.06 112.3949 90)
       (effects (font (size 1.27 1.27)) (justify right))
     )
@@
   (symbol (lib_id "Diode:1N4148") (at 242.57 113.03 90) (unit 1)
     (in_bom yes) (on_board yes)
-    (property "Reference" "D49" (id 0) (at 237.49 112.3949 90)
+    (property "Reference" "D47" (id 0) (at 237.49 112.3949 90)
       (effects (font (size 1.27 1.27)) (justify right))
     )
@@
   (symbol (lib_id "Diode:1N4148") (at 254 113.03 90) (unit 1)
     (in_bom yes) (on_board yes)
-    (property "Reference" "D50" (id 0) (at 248.92 112.3949 90)
+    (property "Reference" "D48" (id 0) (at 248.92 112.3949 90)
       (effects (font (size 1.27 1.27)) (justify right))
     )
@@
       (reference "D45") (unit 1) (value "1N4148") (footprint "Diode_THT:D_DO-35_SOD27_P12.70mm_Horizontal")
     )
-    (path "/2b4cf488-1db9-424e-8864-167bee1ce081"
-      (reference "D46") (unit 1) (value "1N4729") (footprint "Diode_THT:D_DO-41_SOD81_P7.62mm_Horizontal")
-    )
-    (path "/68c3db0c-7e71-4f75-8eba-60f9626e77dc"
-      (reference "D47") (unit 1) (value "1N4729") (footprint "Diode_THT:D_DO-41_SOD81_P7.62mm_Horizontal")
-    )
     (path "/9557c4e1-1779-460e-8a7e-638019af0f88"
-      (reference "D48") (unit 1) (value "1N4148") (footprint "Diode_THT:D_DO-35_SOD27_P12.70mm_Horizontal")
+      (reference "D46") (unit 1) (value "1N4148") (footprint "Diode_THT:D_DO-35_SOD27_P12.70mm_Horizontal")
     )
     (path "/477d73d3-ec9d-4c18-8bd5-c633add13fa7"
-      (reference "D49") (unit 1) (value "1N4148") (footprint "Diode_THT:D_DO-35_SOD27_P12.70mm_Horizontal")
+      (reference "D47") (unit 1) (value "1N4148") (footprint "Diode_THT:D_DO-35_SOD27_P12.70mm_Horizontal")
     )
     (path "/5b1e7fe1-a92e-4f24-a9d3-e86705a90beb"
-      (reference "D50") (unit 1) (value "1N4148") (footprint "Diode_THT:D_DO-35_SOD27_P12.70mm_Horizontal")
+      (reference "D48") (unit 1) (value "1N4148") (footprint "Diode_THT:D_DO-35_SOD27_P12.70mm_Horizontal")
+    )
+    (path "/2b4cf488-1db9-424e-8864-167bee1ce081"
+      (reference "D49") (unit 1) (value "1N4729") (footprint "Diode_THT:D_DO-41_SOD81_P7.62mm_Horizontal")
+    )
+    (path "/68c3db0c-7e71-4f75-8eba-60f9626e77dc"
+      (reference "D50") (unit 1) (value "1N4729") (footprint "Diode_THT:D_DO-41_SOD81_P7.62mm_Horizontal")
     )
     (path "/a24fd230-03ea-471f-b4ba-6e204bed0cee"
